File: ZoeZeroEagle.brd (EAGLE design)
At the start: 65 x 30 mm, 7 parts

Commit message: General update to latest versions
Parts:
- removed E$1, E$2: (no value), con-lstb:MA03-2
- removed E$4: (no value), con-panduit:057-040-1
- removed E$5, E$6, E$7, E$8: (no value), FLYFISH:PIN_W_2
Routing:
- net S$7: track 14.0 -> 300.7 mm, vias 0 -> 37
- net S$4: track 13.5 -> 80.9 mm, vias 0 -> 9
- net S$5: track 65.6 -> 0.00 mm, vias 0 -> 1
- net S$13: track 51.6 -> 0.00 mm
- net S$14: track 43.9 -> 0.00 mm
- net S$3: track 47.0 -> 5.61 mm, vias 0 -> 3
- net S$2: track 38.0 -> 0.00 mm, vias 0 -> 1
- net S$11: track 14.8 -> 0.00 mm
- net S$10: track 12.9 -> 0.00 mm
- net S$17: track 11.8 -> 0.00 mm
- net S$6: track 9.94 -> 0.00 mm, vias 0 -> 1
- net S$9: track 8.89 -> 0.00 mm, vias 0 -> 1
- net S$1: track 0.00 -> 3.81 mm, vias 0 -> 2
Other:
- board size 65 x 30 mm -> 75.2 x 30 mm
- board text added: "3V3"
- board text added: "5V"
- board text added: "CE0"
- board text added: "CE1"
- board text added: "CLK"
- board text added: "G12"
- board text added: "G13"
- board text added: "G16"
- board text added: "G17"
- board text added: "G18"
- board text added: "G19"
- board text added: "G20"
- board text added: "G21"
- board text added: "G22"
- board text added: "G23"
- board text added: "G24"
- board text added: "G25"
- board text added: "G26"
- board text added: "G27"
- board text added: "G5"
- board text added: "G6"
- board text added: "GND"
- board text added: "ID"
- board text added: "MISO"
- board text added: "MOSI"
- board text added: "MOSI=G10 MISO=G9 SCK=G11 CE0=G8 CE1=G7"
- board text added: "RXD"
- board text added: "SC"
- board text added: "SCK"
- board text added: "SCL"
- board text added: "SD"
- board text added: "SDA"
- board text added: "SDA=G2 SCL=G3 CLK=G4 TXD=G14 RXD=G15"
- board text added: "TXD"
