File: RPi0-PCB.brd (EAGLE design)
At the start: 75.2 x 30 mm, 0 parts

Commit message: Tidying up.
Routing:
- net S$8: vias 27 -> 28
Changed lines of the file:
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@@
 <circle x="36.83" y="11.43" radius="0.6" width="0.25" layer="16"/>
 <circle x="39.37" y="11.43" radius="0.6" width="0.25" layer="16"/>
-<circle x="34.29" y="19.05" radius="0.6" width="0.25" layer="16"/>
 <circle x="34.29" y="11.43" radius="0.6" width="0.25" layer="16"/>
 <circle x="36.83" y="19.05" radius="0.6" width="0.25" layer="16"/>
@@
 <circle x="82.55" y="21.59" radius="0.6" width="0.25" layer="16"/>
 <circle x="82.55" y="16.51" radius="0.6" width="0.25" layer="16"/>
+<circle x="34.29" y="19.05" radius="0.6" width="0.25" layer="16"/>
 </plain>
 <attributes>
@@
 <wire x1="80.01" y1="11.43" x2="77.47" y2="13.97" width="0.4064" layer="16"/>
 <wire x1="77.47" y1="13.97" x2="48.26" y2="13.97" width="0.4064" layer="16"/>
+<via x="34.29" y="19.05" extent="1-16" drill="0.9" diameter="1.55"/>
 </signal>
 <signal name="S$59">
